File: pcb/wrangler_v0.kicad_sch (KiCad schematic)
At the start: 60 parts, among them J1 HDMI_A, J2 USB_B_Micro, J3 Conn_01x10, J4 Conn_01x10, SW1 SW_Push, SW2 SW_Push, U1 ICE40UP5K-SG48ITR, U2 W25Q32JVSSIM, U3 AP2127K-3.3, U4 AP2127K-1.2

Commit message: pcb: added CDONE pullup resistor and some silkscreen tweaks
Parts:
- added R25: 2.2k, Resistor_SMD:R_0402_1005Metric, symbol wrangler_v0.0:Device_R
- renumbered SW1 to RESET1, SW2 to SW1
Connections:
- net +3.3V: now also R25.2
- net CDONE: now also R25.1
Other:
- moved on the sheet: RESET1
Changed lines of the file:
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@@
   (junction (at 45.72 33.02) (diameter 0) (color 0 0 0 0)
   )
+  (junction (at 116.84 31.75) (diameter 0) (color 0 0 0 0)
+  )
   (junction (at 382.27 143.51) (diameter 0) (color 0 0 0 0)
   )
@@
     (stroke (width 0) (type default))
   )
+  (wire (pts (xy 127 41.91) (xy 127 45.72))
+    (stroke (width 0) (type default))
+  )
   (wire (pts (xy 140.97 248.92) (xy 140.97 252.73))
     (stroke (width 0) (type default))
@@
     (stroke (width 0) (type default))
   )
+  (wire (pts (xy 59.69 59.69) (xy 59.69 60.96))
+    (stroke (width 0) (type default))
+  )
   (wire (pts (xy 151.13 200.66) (xy 151.13 205.74))
     (stroke (width 0) (type default))
@@
     (stroke (width 0) (type default))
   )
-  (wire (pts (xy 59.69 50.8) (xy 59.69 45.72))
+  (wire (pts (xy 59.69 49.53) (xy 59.69 45.72))
     (stroke (width 0) (type default))
   )
@@
     (stroke (width 0) (type default))
   )
-  (wire (pts (xy 105.41 45.72) (xy 110.49 45.72))
+  (wire (pts (xy 105.41 45.72) (xy 127 45.72))
     (stroke (width 0) (type default))
   )
@@
     (stroke (width 0) (type default))
   )
+  (wire (pts (xy 127 34.29) (xy 127 31.75))
+    (stroke (width 0) (type default))
+  )
   (wire (pts (xy 177.8 251.46) (xy 177.8 255.27))
     (stroke (width 0) (type default))
@@
     (stroke (width 0) (type default))
   )
+  (wire (pts (xy 127 31.75) (xy 116.84 31.75))
+    (stroke (width 0) (type default))
+  )
   (wire (pts (xy 160.02 252.73) (xy 160.02 248.92))
     (stroke (width 0) (type default))
@@
     )
   )
-  (symbol (lib_id "Switch:SW_Push") (at 59.69 55.88 90) (unit 1)
-    (in_bom yes) (on_board yes) (dnp no) (fields_autoplaced)
-    (property "Reference" "SW1" (at 60.96 55.245 90)
+  (symbol (lib_id "Switch:SW_Push") (at 59.69 54.61 90) (unit 1)
+    (in_bom yes) (on_board yes) (dnp no)
+    (property "Reference" "RESET1" (at 60.96 48.26 90)
       (effects (font (size 1.27 1.27)) (justify right))
     )
-    (property "Value" "SW_Push" (at 60.96 57.785 90)
+    (property "Value" "SW_Push" (at 60.96 56.515 90)
       (effects (font (size 1.27 1.27)) (justify right))
     )
-    (property "Footprint" "Button_Switch_SMD:SW_SPST_CK_KXT3" (at 54.61 55.88 0)
+    (property "Footprint" "Button_Switch_SMD:SW_SPST_CK_KXT3" (at 54.61 54.61 0)
       (effects (font (size 1.27 1.27)) hide)
     )
-    (property "Datasheet" "~" (at 54.61 55.88 0)
+    (property "Datasheet" "~" (at 54.61 54.61 0)
       (effects (font (size 1.27 1.27)) hide)
     )
@@
       (project "wrangler_v0"
         (path "/5ef2e1d8-db1b-4f05-b1e6-93d7ceabe469"
-          (reference "SW1") (unit 1)
+          (reference "RESET1") (unit 1)
         )
       )
@@
   (symbol (lib_id "Switch:SW_Push") (at 316.23 48.26 90) (unit 1)
     (in_bom yes) (on_board yes) (dnp no) (fields_autoplaced)
-    (property "Reference" "SW2" (at 317.5 47.625 90)
+    (property "Reference" "SW1" (at 317.5 47.625 90)
       (effects (font (size 1.27 1.27)) (justify right))
     )
@@
       (project "wrangler_v0"
         (path "/5ef2e1d8-db1b-4f05-b1e6-93d7ceabe469"
-          (reference "SW2") (unit 1)
+          (reference "SW1") (unit 1)
         )
       )
@@
         )
       )
+    )
+  )
+  (symbol (lib_id "wrangler_v0.0:Device_R") (at 127 38.1 180) (unit 1)
+    (in_bom yes) (on_board yes) (dnp no)
+    (property "Reference" "R25" (at 128.778 36.9316 0)
+      (effects (font (size 1.27 1.27)) (justify right))
+    )
+    (property "Value" "2.2k" (at 128.778 39.243 0)
+      (effects (font (size 1.27 1.27)) (justify right))
+    )
+    (property "Footprint" "Resistor_SMD:R_0402_1005Metric" (at 128.778 38.1 90)
+      (effects (font (size 1.27 1.27)) hide)
+    )
+    (property "Datasheet" "~" (at 127 38.1 0)
+      (effects (font (size 1.27 1.27)) hide)
+    )
+    (pin "1")
+    (pin "2")
+    (instances
+      (project "wrangler_v0"
+        (path "/5ef2e1d8-db1b-4f05-b1e6-93d7ceabe469"
+          (reference "R25") (unit 1)
+        )
+      )
